File: jtag_2232h.kicad_sch (KiCad schematic)
At the start: 91 parts

Commit message: Another import attempt.
Parts:
- removed CONN_JTAG1: HDR_2x6, jtag_2232h:RCP_1P27_2X6_EDGE, symbol jtag_2232h:root_0_HDR_2x6
- removed CONN_USB1: MICRO_USB_B, jtag_2232h:MICRO_USB_B, symbol jtag_2232h:root_0_MICRO_USB_B
- removed C_EEPROM_VCC1, C_FT_OSC_IN1, C_FT_OSC_OUT1, C_FT_PHY1, C_FT_PLL1, C_FT_REG_OUT1, C_IN_LDO_VCC1, C_OPAMP1, C_OUT_LDO_VCC1, C_VEIO_OUT1: ${ALTIUM_VALUE}, jtag_2232h:M1608, symbol jtag_2232h:root_0_CAP
- removed C_VEIO_CMP1, C_VEIO_FB1: ${ALTIUM_VALUE}, jtag_2232h:M1608, symbol jtag_2232h:root_1_CAP
- removed EPRG_FT_TCK1, EPRG_TCK1, EPRG_TDI1, EPRG_TDO1, EPRG_TMS1, GND1, UDM1, UDN1, UGND1, VBUS1, VCC1, VCORE1, VEIO1, VIIO1: Test_Point, jtag_2232h:TEST_POINT_100, symbol jtag_2232h:root_0_Test_Point
- removed LED_FN1, LED_PWR1: LED_2, jtag_2232h:LEDX2_150X160X55, symbol jtag_2232h:root_3_LED_2
- removed Q_LDO1: BJT_PNP, jtag_2232h:SOT65P210X110_3N_BJT_BEC, symbol jtag_2232h:root_1_BJT_PNP
- removed Q_OV1: BJT_PNP, jtag_2232h:SOT65P210X110_3N_BJT_BEC, symbol jtag_2232h:root_0_BJT_PNP
- removed Q_PWR_LED1: MOSFET_P, jtag_2232h:SOT65P210X110_3N_FET_GSD, symbol jtag_2232h:root_0_MOSFET_P
- removed Q_TPWR1: BJT_NPN, jtag_2232h:SOT95P237X112_3N_BJT_BEC, symbol jtag_2232h:root_0_mirrored_BJT_NPN
- removed R_EIO_BYPASS1, R_EPRG_EN1, R_SPI_DO1, R_VEIO_CMP1, R_VEIO_FB1, R_VEIO_IN1: ${ALTIUM_VALUE}, jtag_2232h:M1608, symbol jtag_2232h:root_0_RES
- removed R_EPRG_TCK_PULL1, R_FT_PHY1, R_FT_PLL1, R_FT_REF1, R_FT_RESET1, R_OUT_LDO_VCC1, R_PWR_LED_PULL1, R_SER_LED_PULL1, R_USB_GND1, R_VEIO_DN1: ${ALTIUM_VALUE}, jtag_2232h:M1608, symbol jtag_2232h:root_1_RES
- removed R_FT_LDO1, R_TPWR1: ${ALTIUM_VALUE}, jtag_2232h:M1608, symbol jtag_2232h:root_2_RES
- removed R_GND_DETECT_PULL1, R_LED_FN1, R_LED_PWR1: ${ALTIUM_VALUE}, jtag_2232h:M1608x2, symbol jtag_2232h:root_1_RES2
- removed R_QBASE1: ${ALTIUM_VALUE}, jtag_2232h:M1608x2, symbol jtag_2232h:root_0_RES2
- removed R_QBASE2: ${ALTIUM_VALUE}, jtag_2232h:M1608x2, symbol jtag_2232h:root_2_RES2
- removed R_SPI1: ${ALTIUM_VALUE}, jtag_2232h:M1608x4, symbol jtag_2232h:root_1_RES4
- removed U_EEPROM1: SPI_EEPROM, jtag_2232h:TSSOP8, symbol jtag_2232h:root_0_mirrored_SPI_EEPROM
- removed U_EPLD1: 5M40Z, jtag_2232h:TSQFP40P900X900X120_HS_64N, symbol jtag_2232h:root_0_5M40Z
- removed U_FTDI1: FT2232H, jtag_2232h:TSQFP50P1200X1200X120_64M, symbol jtag_2232h:root_0_FT2232H
- removed U_LDO_VCC1: LDO_1117, jtag_2232h:SOT89-150P410X160-3N, symbol jtag_2232h:root_0_LDO_1117
- removed U_OPAMP1: MCP6001, jtag_2232h:SOT65P210X110_5N, symbol jtag_2232h:root_0_MCP6001
- removed Y_FTDI1: XTAL_4P, jtag_2232h:XTAL_4P_3P2x2P5, symbol jtag_2232h:root_0_XTAL_4P
- added CONN_JTAG: HDR_2x6, RCP_1P27_2X6_EDGE, symbol jtag_2232h:root_0_HDR_2x6
- added CONN_USB: MICRO_USB_B, MICRO_USB_B, symbol jtag_2232h:root_0_MICRO_USB_B
- added C_EEPROM_VCC, C_FT_OSC_IN, C_FT_OSC_OUT, C_FT_PHY, C_FT_PLL, C_FT_REG_OUT, C_IN_LDO_VCC, C_OPAMP, C_OUT_LDO_VCC, C_VEIO_OUT: ${ALTIUM_VALUE}, M1608, symbol jtag_2232h:root_0_CAP
- added C_VEIO_CMP, C_VEIO_FB: ${ALTIUM_VALUE}, M1608, symbol jtag_2232h:root_1_CAP
- added EPRG_FT_TCK, EPRG_TCK, EPRG_TDI, EPRG_TDO, EPRG_TMS, GND, UDM, UDN, UGND, VBUS, VCC, VCORE, VEIO, VIIO: Test_Point, TEST_POINT_100, symbol jtag_2232h:root_0_Test_Point
- added LED_FN, LED_PWR: LED_2, LEDX2_150X160X55, symbol jtag_2232h:root_3_LED_2
- added Q_LDO: BJT_PNP, SOT65P210X110_3N_BJT_BEC, symbol jtag_2232h:root_1_BJT_PNP
- added Q_OV: BJT_PNP, SOT65P210X110_3N_BJT_BEC, symbol jtag_2232h:root_0_BJT_PNP
- added Q_PWR_LED: MOSFET_P, SOT65P210X110_3N_FET_GSD, symbol jtag_2232h:root_0_MOSFET_P
- added Q_TPWR: BJT_NPN, SOT95P237X112_3N_BJT_BEC, symbol jtag_2232h:root_0_mirrored_BJT_NPN
- added R_EIO_BYPASS, R_EPRG_EN, R_SPI_DO, R_VEIO_CMP, R_VEIO_FB, R_VEIO_IN: ${ALTIUM_VALUE}, M1608, symbol jtag_2232h:root_0_RES
- added R_EPRG_TCK_PULL, R_FT_PHY, R_FT_PLL, R_FT_REF, R_FT_RESET, R_OUT_LDO_VCC, R_PWR_LED_PULL, R_SER_LED_PULL, R_USB_GND, R_VEIO_DN: ${ALTIUM_VALUE}, M1608, symbol jtag_2232h:root_1_RES
- added R_FT_LDO, R_TPWR: ${ALTIUM_VALUE}, M1608, symbol jtag_2232h:root_2_RES
- added R_GND_DETECT_PULL, R_LED_FN, R_LED_PWR: ${ALTIUM_VALUE}, M1608x2, symbol jtag_2232h:root_1_RES2
- added R_QBASE: ${ALTIUM_VALUE}, M1608x2, symbol jtag_2232h:root_2_RES2
- added R_SPI: ${ALTIUM_VALUE}, M1608x4, symbol jtag_2232h:root_1_RES4
- added U_EEPROM: SPI_EEPROM, TSSOP8, symbol jtag_2232h:root_0_mirrored_SPI_EEPROM
- added U_EPLD: 5M40Z, TSQFP40P900X900X120_HS_64N, symbol jtag_2232h:root_0_5M40Z
- added U_FTDI: FT2232H, TSQFP50P1200X1200X120_64M, symbol jtag_2232h:root_0_FT2232H
- added U_LDO_VCC: LDO_1117, SOT89-150P410X160-3N, symbol jtag_2232h:root_0_LDO_1117
- added U_OPAMP: MCP6001, SOT65P210X110_5N, symbol jtag_2232h:root_0_MCP6001
- added Y_FTDI: XTAL_4P, XTAL_4P_3P2x2P5, symbol jtag_2232h:root_0_XTAL_4P
- C_BYP_LDO_V1P8, C_EPLD_V1P8_1, C_EPLD_V1P8_2, C_EPLD_VCC_1, C_EPLD_VCC_2, C_EPLD_VEIO_1, C_EPLD_VEIO_2, C_FT_CORE_1, C_FT_CORE_2, C_FT_CORE_3, C_FT_VCC_1, C_FT_VCC_2, C_FT_VCC_3, C_FT_VCC_4: footprint jtag_2232h:M1608 -> M1608
- D_JTAG_1, D_JTAG_2, D_JTAG_3, D_JTAG_4, D_JTAG_5: footprint jtag_2232h:SOT65P210X110_3N_2DIODE_CC -> SOT65P210X110_3N_2DIODE_CC
- R_JTAG_1, R_JTAG_2: footprint jtag_2232h:M1608x4 -> M1608x4
- R_JTAG_3: footprint jtag_2232h:M1608x2 -> M1608x2
- TVS_JTAG_1, TVS_JTAG_2, TVS_JTAG_3: footprint jtag_2232h:SOT65P210X110_6N -> SOT65P210X110_6N
- U_LDO_V1P8: footprint jtag_2232h:SOT95P255X145_5N -> SOT95P255X145_5N
- V1P8: footprint jtag_2232h:TEST_POINT_100 -> TEST_POINT_100
Connections:
- net EPRG_FT_TCK: now also EPRG_FT_TCK.1, R_EPRG_EN.1, U_FTDI.53 (BCBUS2)
- net EPRG_TCK: now also EPRG_TCK.1, R_EPRG_EN.2, R_EPRG_TCK_PULL.1, U_EPLD.16 (TCK)
- net EPRG_TDI: now also EPRG_TDI.1, U_EPLD.15 (TDI), U_FTDI.57 (BCBUS5)
- net EPRG_TDO: now also EPRG_TDO.1, U_EPLD.17 (TDO), U_FTDI.58 (BCBUS6)
- net EPRG_TMS: now also EPRG_TMS.1, U_EPLD.14 (TMS), U_FTDI.59 (BCBUS7)
- net FT_GPIO_H0: now also U_EPLD.12 (I/O), U_FTDI.26 (ACBUS0)
- net FT_GPIO_H1: now also U_EPLD.11 (I/O), U_FTDI.27 (ACBUS1)
- net FT_GPIO_H2: now also U_EPLD.5 (I/O), U_FTDI.28 (ACBUS2)
- net FT_GPIO_H3: now also U_EPLD.7 (I/O), U_FTDI.29 (ACBUS3)
- net FT_GPIO_H4: now also U_EPLD.9 (I/O), U_FTDI.30 (ACBUS4)
- net FT_GPIO_H5: now also U_EPLD.10 (I/O), U_FTDI.32 (ACBUS5)
- net FT_GPIO_H6: now also U_EPLD.4 (I/O), U_FTDI.33 (ACBUS6)
- net FT_GPIO_H7: now also U_EPLD.3 (I/O), U_FTDI.34 (ACBUS7)
- net FT_GPIO_L0: now also U_EPLD.20 (I/O), U_FTDI.21 (ADBUS4)
- net FT_GPIO_L1: now also U_EPLD.19 (I/O), U_FTDI.22 (ADBUS5)
- net FT_GPIO_L2: now also U_EPLD.18 (I/O), U_FTDI.23 (ADBUS6)
- net FT_JTAG_EN_N: now also Q_PWR_LED.G, R_PWR_LED_PULL.1, U_EPLD.30 (I/O), U_FTDI.60 (PWREN#)
- net FT_JTAG_RTCK: now also U_EPLD.13 (I/O), U_FTDI.24 (ADBUS7)
- net FT_JTAG_TCK: now also U_EPLD.29 (I/O), U_FTDI.16 (ADBUS0)
- net FT_JTAG_TDI: now also U_EPLD.24 (I/O), U_FTDI.17 (ADBUS1)
- net FT_JTAG_TDO: now also U_EPLD.22 (I/O), U_FTDI.18 (ADBUS2)
- net FT_JTAG_TMS: now also U_EPLD.21 (I/O), U_FTDI.19 (ADBUS3)
- net FT_SER_LED: now also R_SER_LED_PULL.1, U_EPLD.64 (I/O), U_FTDI.54 (BCBUS3), U_FTDI.55 (BCBUS4)
- net FT_SER_RXD: now also U_EPLD.1 (I/O), U_FTDI.39 (BDBUS1)
- net FT_SER_TXD: now also U_EPLD.2 (I/O), U_FTDI.38 (BDBUS0)
- net GND: now also CONN_JTAG.5, CONN_JTAG.7, CONN_USB.5 (GND), C_EEPROM_VCC.2, C_FT_OSC_IN.2, C_FT_OSC_OUT.2, C_FT_PHY.2, C_FT_PLL.2, C_FT_REG_OUT.2, C_IN_LDO_VCC.2, C_OPAMP.2, C_VEIO_OUT.2, GND.1, LED_FN.C1, LED_FN.C2, LED_PWR.C1, LED_PWR.C2, Q_OV.C, R_FT_REF.1, R_OUT_LDO_VCC.1, R_USB_GND.1, R_VEIO_DN.1, UGND.1, U_EEPROM.5 (GND), U_EPLD.C (GND), U_FTDI.1 (GND), U_FTDI.10 (AGND), U_FTDI.11 (GND), U_FTDI.13 (TEST), U_FTDI.15 (GND), U_FTDI.25 (GND), U_FTDI.35 (GND), U_FTDI.47 (GND), U_FTDI.5 (GND), U_FTDI.51 (GND), U_LDO_VCC.1 (GND), U_OPAMP.2 (V-), Y_FTDI.2, Y_FTDI.4
- net GND_DETECT: now also CONN_JTAG.11
- net JTAG_RST: now also CONN_JTAG.12
- net JTAG_RTCK: now also CONN_JTAG.9
- net JTAG_TCK: now also CONN_JTAG.6
- net JTAG_TDI: now also CONN_JTAG.10
- net JTAG_TDO: now also CONN_JTAG.8
- net JTAG_TMS: now also CONN_JTAG.4
- net LED_ACT: now also R_LED_FN.3, U_EPLD.31 (I/O)
- net LED_NO_TGT: now also R_LED_FN.4, U_EPLD.32 (I/O)
- net SER_RXD: now also CONN_JTAG.1
- net SER_TXD: now also CONN_JTAG.2
- net USB_DM: now also CONN_USB.2 (D-), UDM.1, U_FTDI.7 (DM)
- net USB_DP: now also CONN_USB.3 (D+), UDN.1, U_FTDI.8 (DP)
- net VCC: now also C_EEPROM_VCC.1, C_OUT_LDO_VCC.1, Q_LDO.E, Q_PWR_LED.S, Q_TPWR.C, R_EPRG_TCK_PULL.2, R_FT_PHY.2, R_FT_PLL.2, R_FT_RESET.2, R_GND_DETECT_PULL.4, R_PWR_LED_PULL.2, R_QBASE.3, R_SER_LED_PULL.2, R_SPI.5, R_SPI.6, R_SPI.7, R_SPI.8, U_EEPROM.6 (ORG), U_EEPROM.8 (VCC), U_EPLD.23 (VCCIO1), U_EPLD.6 (VCCIO1), U_FTDI.20 (VCCIO), U_FTDI.31 (VCCIO), U_FTDI.42 (VCCIO), U_FTDI.50 (VREGIN), U_FTDI.56 (VCCIO), U_LDO_VCC.2 (VOUT), VCC.1
- net VCC_1P8: now also R_FT_LDO.2, U_EPLD.41 (VCCINT), U_EPLD.8 (VCCINT)
- net VCC_EIO: now also C_VEIO_FB.2, C_VEIO_OUT.1, Q_LDO.C, Q_OV.E, R_EIO_BYPASS.2, R_VEIO_FB.2, U_EPLD.39 (VCCIO2), U_EPLD.57 (VCCIO2), VEIO.1
- net VCC_FT_CORE: now also C_FT_REG_OUT.1, R_FT_LDO.1, U_FTDI.12 (VCORE), U_FTDI.37 (VCORE), U_FTDI.49 (VREGOUT), U_FTDI.64 (VCORE), VCORE.1
- net VCC_IO: now also CONN_JTAG.3, R_EIO_BYPASS.1, R_TPWR.1, R_VEIO_DN.2, R_VEIO_IN.1, VIIO.1
- net VCC_VBUS: now also CONN_USB.1 (VBUS), C_IN_LDO_VCC.1, C_OPAMP.1, U_LDO_VCC.3 (VIN), U_OPAMP.5 (V+), VBUS.1
- net at D_JTAG_2.A1, R_JTAG_1.1, TVS_JTAG_1.1 (K): now also U_EPLD.42 (I/O)
- net at D_JTAG_2.A2, R_JTAG_1.3, TVS_JTAG_1.4 (K): now also U_EPLD.43 (I/O)
- net at D_JTAG_4.A1, R_JTAG_2.3, TVS_JTAG_2.4 (K): now also U_EPLD.47 (I/O)
- net at D_JTAG_4.A2, R_JTAG_2.2, TVS_JTAG_2.3 (K): now also U_EPLD.46 (I/O)
- net at D_JTAG_3.A1, R_JTAG_1.4, TVS_JTAG_1.6 (K): now also U_EPLD.44 (I/O)
- net at D_JTAG_3.A2, R_JTAG_2.1, TVS_JTAG_2.1 (K): now also U_EPLD.45 (I/O)
- net at D_JTAG_1.A2, R_JTAG_1.2, TVS_JTAG_1.3 (K): now also R_GND_DETECT_PULL.1, U_EPLD.33 (I/O)
- net at D_JTAG_5.A1, R_JTAG_2.4, TVS_JTAG_2.6 (K): now also U_EPLD.48 (I/O)
- net at D_JTAG_5.A2, R_JTAG_3.1, TVS_JTAG_3.6 (K): now also U_EPLD.49 (I/O)
- new net: LED_FN.A1, R_LED_FN.1
- new net: LED_PWR.A1, R_LED_PWR.1
- new net: Q_PWR_LED.D, R_LED_PWR.4
- new net: Q_LDO.B, R_QBASE.4
- new net: Q_TPWR.B, R_TPWR.2
- new net: Q_TPWR.E, R_LED_PWR.3
- new net: C_FT_PHY.1, R_FT_PHY.1, U_FTDI.4 (VPHY)
- new net: R_VEIO_CMP.1, R_VEIO_IN.2, U_OPAMP.4 (-)
- new net: C_VEIO_CMP.1, R_VEIO_CMP.2
- new net: R_FT_RESET.1, U_FTDI.14 (RESET#)
- new net: C_FT_OSC_IN.1, U_FTDI.2 (OSCI), Y_FTDI.1
- new net: C_FT_OSC_OUT.1, U_FTDI.3 (OSCO), Y_FTDI.3
- new net: R_FT_REF.2, U_FTDI.6 (REF)
- new net: R_SPI.2, R_SPI_DO.2, U_EEPROM.3 (D_IN), U_FTDI.61 (EEDATA)
- new net: R_SPI.3, U_EEPROM.2 (SCLK), U_FTDI.62 (EECLK)
- new net: R_SPI.4, U_EEPROM.1 (CS_N), U_FTDI.63 (EECS)
- new net: C_FT_PLL.1, R_FT_PLL.1, U_FTDI.9 (VPLL)
- new net: C_VEIO_CMP.2, R_QBASE.1, U_OPAMP.1 (Vout)
- new net: R_SPI_DO.1, U_EEPROM.4 (D_OUT)
- new net: Q_OV.B, R_QBASE.2
- new net: CONN_USB.SHELL, R_USB_GND.2
- new net: LED_PWR.A2, R_LED_PWR.2
- new net: LED_FN.A2, R_LED_FN.2
- new net: C_VEIO_FB.1, R_VEIO_FB.1, U_OPAMP.3 (+)
- new net: C_OUT_LDO_VCC.2, R_OUT_LDO_VCC.2

Commit message: Cleared all DRCs, mostly fixed up library.
Parts:
- added LOGO1: ~, jtag_2232h:MC_logo_micro, symbol jtag_2232h:MC_logo
- renumbered CONN_JTAG to CONN_JTAG1, CONN_USB to CONN_USB1, C_EEPROM_VCC to C_EEPROM_VCC1, C_FT_OSC_IN to C_FT_OSC_IN1, C_FT_OSC_OUT to C_FT_OSC_OUT1, C_FT_PHY to C_FT_PHY1, C_FT_PLL to C_FT_PLL1, C_FT_REG_OUT to C_FT_REG_OUT1, C_IN_LDO_VCC to C_IN_LDO_VCC1, C_OPAMP to C_OPAMP1, C_OUT_LDO_VCC to C_OUT_LDO_VCC1, C_VEIO_CMP to C_VEIO_CMP1, C_VEIO_FB to C_VEIO_FB1, C_VEIO_OUT to C_VEIO_OUT1, EPRG_FT_TCK to EPRG_FT_TCK1, EPRG_TCK to EPRG_TCK1, EPRG_TDI to EPRG_TDI1, EPRG_TDO to EPRG_TDO1, EPRG_TMS to EPRG_TMS1, GND to GND1, LED_FN to LED_FN1, LED_PWR to LED_PWR1, Q_LDO to Q_LDO1, Q_OV to Q_OV1, Q_PWR_LED to Q_PWR_LED1, Q_TPWR to Q_TPWR1, R_EIO_BYPASS to R_EIO_BYPASS1, R_EPRG_EN to R_EPRG_EN1, R_EPRG_TCK_PULL to R_EPRG_TCK_PULL1, R_FT_LDO to R_FT_LDO1, R_FT_PHY to R_FT_PHY1, R_FT_PLL to R_FT_PLL1, R_FT_REF to R_FT_REF1, R_FT_RESET to R_FT_RESET1, R_GND_DETECT_PULL to R_GND_DETECT_PULL1, R_LED_FN to R_LED_FN1, R_LED_PWR to R_LED_PWR1, R_OUT_LDO_VCC to R_OUT_LDO_VCC1, R_PWR_LED_PULL to R_PWR_LED_PULL1, R_QBASE to R_QBASE1, R_SER_LED_PULL to R_SER_LED_PULL1, R_SPI to R_SPI1, R_SPI_DO to R_SPI_DO1, R_TPWR to R_TPWR1, R_USB_GND to R_USB_GND1, R_VEIO_CMP to R_VEIO_CMP1, R_VEIO_DN to R_VEIO_DN1, R_VEIO_FB to R_VEIO_FB1, R_VEIO_IN to R_VEIO_IN1, UDM to UDM1, UDN to UDN1, UGND to UGND1, U_EEPROM to U_EEPROM1, U_EPLD to U_EPLD1, U_FTDI to U_FTDI1, U_LDO_VCC to U_LDO_VCC1, U_OPAMP to U_OPAMP1, VBUS to VBUS1, VCC to VCC1, VCORE to VCORE1, VEIO to VEIO1, VIIO to VIIO1, Y_FTDI to Y_FTDI1

Commit message: Now using USB-C connector.
Also using much more KiCAD-like components.
Parts:
- removed CONN_USB1: MICRO_USB_B, MICRO_USB_B, symbol jtag_2232h:root_0_MICRO_USB_B
- removed D_JTAG_1, D_JTAG_2, D_JTAG_3, D_JTAG_4, D_JTAG_5: DIODE_2_CC, SOT65P210X110_3N_2DIODE_CC, symbol jtag_2232h:root_1_DIODE_2_CC
- removed Q_LDO1: BJT_PNP, SOT65P210X110_3N_BJT_BEC, symbol jtag_2232h:root_1_BJT_PNP
- removed Q_OV1: BJT_PNP, SOT65P210X110_3N_BJT_BEC, symbol jtag_2232h:root_0_BJT_PNP
- removed Q_PWR_LED1: MOSFET_P, SOT65P210X110_3N_FET_GSD, symbol jtag_2232h:root_0_MOSFET_P
- removed Q_TPWR1: BJT_NPN, SOT95P237X112_3N_BJT_BEC, symbol jtag_2232h:root_0_mirrored_BJT_NPN
- removed R_OUT_LDO_VCC1: ${ALTIUM_VALUE}, M1608, symbol jtag_2232h:root_1_RES
- removed U_OPAMP1: MCP6001, SOT65P210X110_5N, symbol jtag_2232h:root_0_MCP6001
- added D2, D3, D4, D5, D6: BAV70W, Package_TO_SOT_SMD:SOT-323_SC-70, symbol Diode:BAV70W
- added J1: USB_C_Receptacle_USB2.0_14P, Connector_USB:USB_C_Receptacle_HRO_TYPE-C-31-M-12, symbol Connector:USB_C_Receptacle_USB2.0_14P
- added Q1: BC848W, Package_TO_SOT_SMD:SOT-323_SC-70, symbol Transistor_BJT:BC848W
- added Q2, Q3: BC807W, Package_TO_SOT_SMD:SOT-323_SC-70, symbol Transistor_BJT:BC807W
- added Q4: BSS84AKW, Package_TO_SOT_SMD:SOT-323_SC-70, symbol Transistor_FET:BSS84
- added TVS_JTAG_4: ESD5V0S4US, Package_TO_SOT_SMD:SOT-363_SC-70-6, symbol jtag_2232h:root_0_SMS05T1
- added U1: MCP6001x-LT, Package_TO_SOT_SMD:SOT-353_SC-70-5, symbol Amplifier_Operational:MCP6001x-LT
- C_BYP_LDO_V1P8, C_EEPROM_VCC1, C_EPLD_V1P8_1, C_EPLD_V1P8_2, C_EPLD_VCC_1, C_EPLD_VCC_2, C_EPLD_VEIO_1, C_EPLD_VEIO_2, C_FT_CORE_1, C_FT_CORE_2, C_FT_CORE_3, C_FT_OSC_IN1, C_FT_OSC_OUT1, C_FT_PHY1, C_FT_PLL1, C_FT_REG_OUT1, C_FT_VCC_1, C_FT_VCC_2, C_FT_VCC_3, C_FT_VCC_4, C_IN_LDO_VCC1, C_OPAMP1, C_OUT_LDO_VCC1, C_VEIO_CMP1, C_VEIO_FB1, C_VEIO_OUT1: footprint M1608 -> Capacitor_SMD:C_0603_1608Metric_Pad1.08x0.95mm_HandSolder
- LOGO1: footprint jtag_2232h:MC_logo_micro -> jtag_ft2232h:MC_logo_micro
- R_EIO_BYPASS1, R_EPRG_EN1, R_EPRG_TCK_PULL1, R_FT_LDO1, R_FT_PHY1, R_FT_PLL1, R_FT_REF1, R_FT_RESET1, R_PWR_LED_PULL1, R_SER_LED_PULL1, R_SPI_DO1, R_TPWR1, R_USB_GND1, R_VEIO_CMP1, R_VEIO_DN1, R_VEIO_FB1, R_VEIO_IN1: footprint M1608 -> Resistor_SMD:R_0603_1608Metric_Pad0.98x0.95mm_HandSolder
- R_GND_DETECT_PULL1, R_JTAG_3, R_LED_FN1, R_LED_PWR1, R_QBASE1: footprint M1608x2 -> Resistor_SMD:R_Array_Convex_2x0603
- R_JTAG_1, R_JTAG_2, R_SPI1: footprint M1608x4 -> Resistor_SMD:R_Array_Convex_4x0603
- TVS_JTAG_1, TVS_JTAG_2, TVS_JTAG_3: footprint SOT65P210X110_6N -> Package_TO_SOT_SMD:SOT-363_SC-70-6
- U_EEPROM1: footprint TSSOP8 -> Package_SO:TSSOP-8_4.4x3mm_P0.65mm
- U_FTDI1: footprint TSQFP50P1200X1200X120_64M -> Package_QFP:LQFP-64_10x10mm_P0.5mm
- U_LDO_V1P8: footprint SOT95P255X145_5N -> Package_TO_SOT_SMD:SOT-23-5
- U_LDO_VCC1: footprint SOT89-150P410X160-3N -> Package_TO_SOT_SMD:SOT-89-3_Handsoldering
Connections:
- net FT_JTAG_EN_N: now also Q4.1 (G)
- net GND: now also C_OUT_LDO_VCC1.2, J1.A1 (GND), J1.A12 (GND), J1.B1 (GND), J1.B12 (GND), Q2.3 (C), TVS_JTAG_4.2 (A), TVS_JTAG_4.5 (A), U1.2 (V-)
- net GND_DETECT: now also R_JTAG_1.6; no longer R_JTAG_1.7
- net JTAG_RST: now also R_JTAG_1.5; no longer R_JTAG_1.8
- net JTAG_RTCK: now also R_JTAG_1.8; no longer R_JTAG_1.5
- net JTAG_TCK: now also R_JTAG_2.6; no longer R_JTAG_2.7
- net JTAG_TDI: now also R_JTAG_1.7; no longer R_JTAG_1.6
- net JTAG_TDO: now also R_JTAG_2.5; no longer R_JTAG_2.8
- net JTAG_TMS: now also R_JTAG_2.7; no longer R_JTAG_2.6
- net LED_ACT: now also R_LED_FN1.4; no longer R_LED_FN1.3
- net LED_NO_TGT: now also R_LED_FN1.3; no longer R_LED_FN1.4
- net SER_RXD: now also R_JTAG_3.1; no longer R_JTAG_3.4
- net SER_TXD: now also R_JTAG_2.8; no longer R_JTAG_2.5
- net USB_DM: now also J1.A7 (D-), J1.B7 (D-), TVS_JTAG_4.3 (K)
- net USB_DP: now also J1.A6 (D+), J1.B6 (D+), TVS_JTAG_4.1 (K)
- net VCC: now also R_GND_DETECT_PULL1.1, R_QBASE1.4, D2.3 (K), Q1.3 (C), Q3.2 (E), Q4.2 (S); no longer R_GND_DETECT_PULL1.4, R_QBASE1.3
- net VCC_EIO: now also D3.3 (K), D4.3 (K), D5.3 (K), D6.3 (K), Q2.2 (E), Q3.3 (C)
- net VCC_VBUS: now also J1.A4 (VBUS), J1.A9 (VBUS), J1.B4 (VBUS), J1.B9 (VBUS), TVS_JTAG_4.4 (K), U1.5 (V+)
- net at R_LED_FN1.1: now also LED_FN1.A2; no longer LED_FN1.A1
- net at R_LED_PWR1.1: now also LED_PWR1.A2; no longer LED_PWR1.A1
- net at R_LED_PWR1.4: now also Q1.2 (E)
- net at R_TPWR1.2: now also Q1.1 (B)
- net at R_LED_PWR1.3: now also Q4.3 (D)
- net at R_VEIO_CMP1.1, R_VEIO_IN1.2: now also U1.4 (-)
- net at R_SPI_DO1.2, U_EEPROM1.3 (D_IN), U_FTDI1.61 (EEDATA): now also R_SPI1.3; no longer R_SPI1.2
- net at U_EEPROM1.2 (SCLK), U_FTDI1.62 (EECLK): now also R_SPI1.2; no longer R_SPI1.3
- net at U_EEPROM1.1 (CS_N), U_FTDI1.63 (EECS): now also R_SPI1.1; no longer R_SPI1.4
- net at TVS_JTAG_1.1 (K), U_EPLD1.42 (I/O): now also R_JTAG_1.4, D3.1 (A); no longer R_JTAG_1.1
- net at TVS_JTAG_1.3 (K), U_EPLD1.33 (I/O): now also R_GND_DETECT_PULL1.4, R_JTAG_1.3, D2.2 (A); no longer R_GND_DETECT_PULL1.1, R_JTAG_1.2
- net at TVS_JTAG_1.4 (K), U_EPLD1.43 (I/O): now also R_JTAG_1.2, D3.2 (A); no longer R_JTAG_1.3
- net at TVS_JTAG_1.6 (K), U_EPLD1.44 (I/O): now also R_JTAG_1.1, D4.1 (A); no longer R_JTAG_1.4
- net at C_VEIO_CMP1.2: now also R_QBASE1.2, U1.1; no longer R_QBASE1.1
- net at TVS_JTAG_2.4 (K), U_EPLD1.47 (I/O): now also R_JTAG_2.2, D5.1 (A); no longer R_JTAG_2.3
- net at TVS_JTAG_2.6 (K), U_EPLD1.48 (I/O): now also R_JTAG_2.1, D6.1 (A); no longer R_JTAG_2.4
- net at TVS_JTAG_3.6 (K), U_EPLD1.49 (I/O): now also R_JTAG_3.4, D6.2 (A); no longer R_JTAG_3.1
- net at TVS_JTAG_2.1 (K), U_EPLD1.45 (I/O): now also R_JTAG_2.4, D4.2 (A); no longer R_JTAG_2.1
- net at R_USB_GND1.2: now also J1.S1 (SHIELD)
- net at R_LED_PWR1.2: now also LED_PWR1.A1; no longer LED_PWR1.A2
- net at R_LED_FN1.2: now also LED_FN1.A1; no longer LED_FN1.A2
- net at C_VEIO_FB1.1, R_VEIO_FB1.1: now also U1.3 (+)
- net at TVS_JTAG_2.3 (K), U_EPLD1.46 (I/O): now also R_JTAG_2.3, D5.2 (A); no longer R_JTAG_2.2
- new net: Q3.1 (B), R_QBASE1.3
- new net: Q2.1 (B), R_QBASE1.1
- no-connect marks 10 -> 9
Other:
- moved on the sheet: R_JTAG_1A, R_JTAG_1B, R_JTAG_1C, R_JTAG_1D, R_JTAG_2A, R_JTAG_2B, R_JTAG_2C, R_JTAG_2D, R_LED_FN1A, R_LED_FN1B, R_LED_PWR1A, R_LED_PWR1B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
